File: schematics/synth_revC.sch (EAGLE design)
At the start: 270 parts, among them IC1 74AHC1G125, IC2 MCP73831/OT, IC3 74AHC1G125, IC4 74AHC1G125, J100 PINHEAD-2x5-P1.27, SW1 SPST_TACT-KMR2, U1 TLV274IPWR, U10 DMMT3906W-7-F, U11 DMMT3906W-7-F, U12 TLV7101828DSER, U13 SPX3819M5-L-3-3, U14 TLV274IPWR, U15 TLV274IPWR, U16 DMMT3906W-7-F, U17 DMMT3906W-7-F, U18 TLV274IPWR, U2 DMMT3906W-7-F, U21 DMMT3906W-7-F, U22 DMMT3906W-7-F, U24 DMMT3906W-7-F, U25 DMMT3906W-7-F, U27 DMMT3906W-7-F, U28 DMMT3906W-7-F, U3 DMMT3906W-7-F, U30 DMMT3906W-7-F, U31 DMMT3906W-7-F, U4 TLV274IPWR, U5 AD7147ACPZ-1500RL7, U6 DMMT3906W-7-F, U7 DMMT3906W-7-F, U8 TLV274IPWR, U9 TLV274IPWR, X2 32.768, X3 microUSB, X4 microsd

Commit message: DM: not sure
Parts:
- removed RN1: 33, resistor-dil:4R-N0603-ARC
- removed SJ1: (no value), microbuilder:SOLDERJUMPERCLOSED
- added C82: 1u, rcl:C-EUC0603
- added D3: (no value), diode:DIODE-SOD123
- added FB3: (no value), microbuilder:FERRITE0805
- added R72, R73: 10k, rcl:R-US_R0603
- added R74: 63.5k, rcl:R-US_R0603
- added R75: 20k, rcl:R-US_R0603
- added U$19: LM4819MMX, deanParts:LM4819MMX
- C21: value .1u -> 10u
- C60: value 100u -> 1u; device rcl:CPOL-USC -> rcl:C-EUC0603
- R12: value 2.2k -> 10k; device adafruit:R-US_R0603 -> rcl:R-US_R0603
- R66: value 100 -> 20k; device adafruit:R-US_R0805 -> rcl:R-US_R0603
- R68: value 100k -> 10k
- R69: value 100k -> 1k
- U13: value SPX3819M5-L-3-3 -> TLV2471IDBVT; device Exar_By_element14_Batch_1:SPX3819M5-L-3-3 -> deanParts:TLV2471IDBVT
- U5: value AD7147ACPZ-1500RL7 -> mic5225-3.3; device Analog Devices_By_element14_Batch_1:AD7147ACPZ-1500RL7 -> microbuilder:VREG_SOT23-5
Connections:
- removed net CIN0: U5.CIN0
- removed net CIN1: U5.CIN1
- removed net CIN10: U5.CIN10
- removed net CIN11: U5.CIN11
- removed net CIN12: U5.CIN12
- removed net CIN2: U5.CIN2
- removed net CIN3: U5.CIN3
- removed net CIN4: U5.CIN4
- removed net CIN5: U5.CIN5
- removed net CIN6: U5.CIN6
- removed net CIN7: U5.CIN7
- removed net CIN8: U5.CIN8
- removed net CIN9: U5.CIN9
- removed net CT_CS: RN1D.1, SAMD21.PB02/I2/AIN10/SERCOM5.0
- removed net CT_INT: R12.2, SAMD21.PA06/EINT6/AIN6/SERCOM0.2, U5.~INT
- removed net CUTOFF_AUX: JP1.34, R63.2, SJ1.2
- removed net N$158: FB1.P$1, R66.2
- removed net N$204: JP1.5
- removed net N$223: JP1.4
- new net A5: JP1.4, SAMD21.PB02/I2/AIN10/SERCOM5.0
- new net AUDIO_OUT1: C60.1, U$19.BYPASS, U$19.VIN+
- new net D8: JP1.22, SAMD21.PA06/EINT6/AIN6/SERCOM0.2
- new net GND2: C6.-, C61.2, C63.2, C65.2, C67.2, C72.2, C75.2, C76.2, C79.2, C82.2, FB3.P$2, JP1.37, R15.1, R190.2, R21.1, R27.1, R37.1, R49.1, R53.1, R6.1, R62.1, U$19.GND, U$19.SHUTDOWN, U13G$2.V-, U14G$5.V-, U15G$5.V-, U18G$5.V-, U1G$5.V-, U4G$5.V-, U8G$5.V-, U9G$5.V-
- new net N$26: C21.1, R73.2, U13G$1.+IN
- new net OUT: 3.3V.TP, C29.1, C31.1, U5.OUT
- new net VIN: C5.1, D1.C, D3.C, FB2.P$1, JP1.5
- net $P9999: now also C7.1, U5.IN; no longer C60.+, U13.VIN
- net +3.3V: now also C82.1, U$19.VDD, U13G$2.V+; no longer 3.3V.TP, C21.1, C29.1, C31.1, C8.1, R12.1, U13.VOUT, U5.VCC, U5.VDRIVE
- net 4P: now also C21.2
- net AGND: now also C60.2, R12.1, R73.1; no longer CN3.P$1
- net AUDIO_OUT: now also R66.2; no longer CN3.P$2, CN3.P$5
- net GND: now also C7.2, CN2.1, FB3.P$1; no longer C21.2, C6.-, C60.-, C61.2, C63.2, C65.2, C67.2, C7.1, C72.2, C75.2, C76.2, C79.2, CN2.2, JP1.37, R15.1, R190.2, R21.1, R27.1, R37.1, R49.1, R53.1, R6.1, R62.1, U13.GND, U14G$5.V-, U15G$5.V-, U18G$5.V-, U1G$5.V-, U4G$5.V-, U5.EP, U8G$5.V-, U9G$5.V-
- net MISO: no longer RN1A.1
- net MOSI: no longer RN1B.1
- net N$153: now also R74.1
- net N$159: now also FB1.P$1; no longer R66.1
- net N$16: now also U5.EN; no longer U13.EN
- net N$33: now also R12.2, R72.1, U13G$1.-IN; no longer RN1C.2, U5.SCLK
- net N$34: now also R72.2, R74.2, U13G$1.OUT; no longer RN1D.2, U5.~CS
- net N$42: now also CN3.P$2, CN3.P$5, U$19.VO2; no longer C7.2, U5.BIAS
- net N$44: now also R66.1, R75.2, U$19.VIN-; no longer RN1A.2, U5.SDO
- net N$46: now also CN3.P$1, R75.1, U$19.VO1; no longer RN1B.2, U5.SDI
- net PWM_CUTOFF: now also JP1.34, R63.2; no longer SJ1.1
- net SCK: no longer RN1C.1
- net VBAT: now also C8.1, CN2.2; no longer CN2.1
- net VBUS: now also D3.A; no longer C5.1, D1.C, FB2.P$1
Other:
- note removed: "TODO: FIX POLARITY"
- moved on the sheet: C30, C51, C81, C89, CN2, CN3, FB1, IC2, L, LED1, R164, R66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
